Commit message: feat: ML3.1 — aparência do robô, guia de operação e reconciliação de docs
Wrapper fino sobre o TurtleBot 4 upstream (nav2_minimal_tb4_description) no
lugar da montagem peça a peça por mesh, que foi tentada e abandonada: cada mesh
carrega origem e rotação próprias, então reparentar as peças numa árvore de
links nossa espalhava o conjunto.

A causa real do "robô com partes separadas" era o RViz, não o modelo. O
nav2_default_view.rviz do nav2_bringup vem com RobotModel Enabled:false e TF
desenhando 33 triedros rotulados — indistinguível, a olho, de um robô mal
montado. Duas trocas de modelo foram gastas antes de alguém abrir a config.
Daí demo_bringup/rviz/demo_view.rviz.

Também: três pendências do ML3 (world default inexistente, comentários que
afirmavam o oposto da armadilha de escopo de tópicos, xacro_args/use_meshes),
weld_fixed_joints.py, e dois documentos em docs/.

Reconciliação de documentação para o layout de compose do ML3.5: o eixo passa a
ser máquina (host/module), não modo. compose/{learn,emul,target}.yaml estavam
vazios e foram removidos; CLAUDE.md e .ai/CLAUDE.md atualizados. O modo emul cai
junto — imagens arm64 seguem construídas sob QEMU, sem compose dedicado.

Verificado: colcon build limpo (6 pacotes), colcon test 39 testes 0 falhas.
NÃO verificado: confirmação visual em RViz2/Gazebo com GUI (exige sessão
gráfica interativa) — pendente do operador.

File: ros2_ws/src/demo_description/urdf/demo_robot.urdf.xacro (robot description, xacro)
@@ -3,170 +3,121 @@
   demo_robot — differential-drive robot for the Aquila AM69 ROS 2 demo.
   Runs on: x86 host only (Gazebo/RViz2 never run on the module — CLAUDE.md rule 1).
-  Frame tree produced by this model (via robot_state_publisher):
-      base_footprint                 ground projection, Nav2's robot_base_frame
-        └── base_link                chassis origin, at wheel-axle height
-              ├── laser_frame
-              ├── camera_link
-              ├── left_wheel_link
-              ├── right_wheel_link
-              └── caster_wheel_link
-  odom -> base_footprint is published by the Gazebo DiffDrive plugin (ML3).
-  map  -> odom          is published by Nav2's amcl (ML3).
-  Neither is this file's job. See README.md for the full TF ownership table.
-  Every dimension below is a xacro arg — nothing is hardcoded. Override at
-  launch time, e.g.:
-      xacro demo_robot.urdf.xacro wheel_separation:=0.40
+  ============================ WHY THIS IS A WRAPPER ============================
+  This file used to hand-assemble the robot from individual TurtleBot 4 meshes
+  (shell.dae, tower_standoff.dae, rplidar.dae, ...) with offsets derived by
+  measuring mesh bounding boxes. That approach was abandoned: every mesh carries
+  its own internal origin and rotation, so re-parenting the parts onto our own
+  link tree scattered them visibly, and each re-measurement fixed one part while
+  moving another.
+  We now include the upstream, fully-assembled model:
+      /opt/ros/jazzy/share/nav2_minimal_tb4_description/urdf/standard/turtlebot4.urdf.xacro
+  It is maintained by the Nav2 team, its offsets are correct by construction, and
+  it ships the DiffDrive + JointStatePublisher system plugins plus a richer sensor
+  set (RPLIDAR A1, OAK-D RGBD stereo camera, IMU) than we had.
+  Do NOT re-add per-part meshes here. If the robot looks wrong, fix it upstream
+  or override a joint below — do not rebuild the assembly.
+  ========================== WHAT THIS WRAPPER CHANGES ==========================
+  Upstream is a TurtleBot 4, not "our" robot, so three things need overriding to
+  satisfy this project's invariants. Each is done by re-declaring the element
+  AFTER the include — xacro's last-definition-wins applies to <gazebo> blocks.
+  1. gz topic names. Upstream's DiffDrive uses /cmd_vel + /odom and its sensors
+     use /scan and /rgbd_camera/*. Those are already short/unscoped names, which
+     is what demo_simulation/config/bridge_warehouse.yaml needs, so they are kept
+     as-is. See that file for the mapping to the /demo/* contract.
+  2. Odometry frame. Upstream's DiffDrive publishes odom -> base_link, and its
+     child_frame_id is HARDCODED in
+     nav2_minimal_tb4_description/urdf/icreate/create3.urdf.xacro with no xacro
+     arg to override it.
+     Re-declaring the plugin here does NOT override it. xacro does not merge or
+     replace <gazebo> blocks — it concatenates them, so the expanded URDF ends up
+     with TWO DiffDrive plugins driving the same two joints. That was tried and
+     rejected. Count the plugin ELEMENTS, not text matches — any grep also hits
+     this very comment. test_exactly_one_of_each_gz_system_plugin does it properly.
+     So the frame is reconciled on the Nav2 side instead: robot_base_frame is
+     base_link in demo_navigation/config/nav2_params.yaml.
+     This is safe, not a compromise. The TF tree direction differs from our old
+     model:
+         ours (before): base_footprint (root) -> base_link
+         upstream:      base_link (root)      -> base_footprint
+     and base_footprint_joint is a fixed IDENTITY transform (xyz 0 0 0, rpy 0 0 0),
+     so odom -> base_link and odom -> base_footprint are numerically the same
+     edge. Nav2 gains nothing from base_footprint here and both frames sit at the
+     same height, because upstream places base_link at ground level rather than at
+     wheel-axle height like our old model did.
+  3. Velocity limits. Upstream clamps to 0.5 m/s and 2.0 rad/s inside the plugin.
+     Nav2's controller limits must not exceed these or the controller commands a
+     speed the simulator silently refuses to reach, which reads as a tuning
+     problem. They are matched in nav2_params.yaml.
+  Override at launch time, e.g.:
+      xacro demo_robot.urdf.xacro robot_name:=demo_robot
 -->
 <robot xmlns:xacro="http://www.ros.org/wiki/xacro" name="demo_robot">
-  <!-- ============================ Parameters ============================ -->
-  <!-- Identity. Must match the -name passed to `ros_gz_sim create` in ML3,
-       because the DiffDrive plugin's gz topics are scoped /model/<name>/... -->
+  <!-- Identity. Must match the -name passed to `ros_gz_sim create`. -->
   <xacro:arg name="robot_name" default="demo_robot"/>
-  <!-- Chassis -->
-  <xacro:arg name="chassis_length" default="0.40"/>
-  <xacro:arg name="chassis_width"  default="0.30"/>
-  <xacro:arg name="chassis_height" default="0.15"/>
-  <xacro:arg name="chassis_mass"   default="6.0"/>
-  <!-- Driven wheels. wheel_separation is THE critical DiffDrive parameter:
-       it must equal the actual track width or odometry rotation will be wrong. -->
-  <xacro:arg name="wheel_radius"        default="0.05"/>
-  <xacro:arg name="wheel_width"         default="0.03"/>
-  <xacro:arg name="wheel_separation"    default="0.35"/>
-  <xacro:arg name="wheel_mass"          default="0.5"/>
-  <xacro:arg name="wheel_base_offset_x" default="-0.05"/>
-  <!-- Passive caster -->
-  <xacro:arg name="caster_radius" default="0.025"/>
-  <xacro:arg name="caster_mass"   default="0.2"/>
-  <!-- Lidar -->
-  <xacro:arg name="lidar_offset_x" default="0.15"/>
-  <xacro:arg name="lidar_offset_z" default="0.10"/>
-  <xacro:arg name="lidar_samples"  default="360"/>
-  <xacro:arg name="lidar_range_max" default="12.0"/>
-  <!-- Camera -->
-  <xacro:arg name="camera_offset_x" default="0.18"/>
-  <xacro:arg name="camera_offset_z" default="0.05"/>
-  <xacro:arg name="camera_width"    default="640"/>
-  <xacro:arg name="camera_height"   default="480"/>
-  <!-- Bind args to properties so macros can do arithmetic on them. -->
-  <xacro:property name="robot_name"          value="$(arg robot_name)"/>
-  <xacro:property name="chassis_length"      value="$(arg chassis_length)"/>
-  <xacro:property name="chassis_width"       value="$(arg chassis_width)"/>
-  <xacro:property name="chassis_height"      value="$(arg chassis_height)"/>
-  <xacro:property name="chassis_mass"        value="$(arg chassis_mass)"/>
-  <xacro:property name="wheel_radius"        value="$(arg wheel_radius)"/>
-  <xacro:property name="wheel_width"         value="$(arg wheel_width)"/>
-  <xacro:property name="wheel_separation"    value="$(arg wheel_separation)"/>
-  <xacro:property name="wheel_mass"          value="$(arg wheel_mass)"/>
-  <xacro:property name="wheel_base_offset_x" value="$(arg wheel_base_offset_x)"/>
-  <xacro:property name="caster_radius"       value="$(arg caster_radius)"/>
-  <xacro:property name="caster_mass"         value="$(arg caster_mass)"/>
-  <xacro:property name="lidar_offset_x"      value="$(arg lidar_offset_x)"/>
-  <xacro:property name="lidar_offset_z"      value="$(arg lidar_offset_z)"/>
-  <xacro:property name="lidar_samples"       value="$(arg lidar_samples)"/>
-  <xacro:property name="lidar_range_max"     value="$(arg lidar_range_max)"/>
-  <xacro:property name="camera_offset_x"     value="$(arg camera_offset_x)"/>
-  <xacro:property name="camera_offset_z"     value="$(arg camera_offset_z)"/>
-  <xacro:property name="camera_width"        value="$(arg camera_width)"/>
-  <xacro:property name="camera_height"       value="$(arg camera_height)"/>
-  <!-- ============================== Includes ============================ -->
-  <xacro:include filename="$(find demo_description)/urdf/_materials.xacro"/>
-  <xacro:include filename="$(find demo_description)/urdf/_inertia.xacro"/>
-  <xacro:include filename="$(find demo_description)/urdf/_wheel.xacro"/>
-  <xacro:include filename="$(find demo_description)/urdf/_sensors.xacro"/>
-  <!-- ============================== Links =============================== -->
   <!--
-    base_footprint is the ROOT and the parent of base_link, following the
-    standard ROS convention (same as turtlebot3 / nav2_minimal_tb4). It is a
-    massless, collision-free frame at ground level; Nav2 uses it as
-    robot_base_frame so that costmap footprints sit on the floor plane.
+    Accepted and intentionally ignored.
+    The old hand-built model had a use_meshes:=false path that fell back to
+    primitives for renderer-less arm64 images. Upstream is mesh-only, so there is
+    nothing to switch. This arg is kept ONLY so that existing launch files and
+    documented commands that pass use_meshes:=... keep working instead of dying
+    on an "unknown argument" error.
+    Nothing about the module side depends on it: no OGRE 2 application (Gazebo,
+    RViz2) ever runs on the Aquila, so the module never renders this model at all.
   -->
-  <link name="base_footprint"/>
-  <link name="base_link">
-    <visual>
-      <origin xyz="0 0 0" rpy="0 0 0"/>
-      <geometry>
-        <box size="${chassis_length} ${chassis_width} ${chassis_height}"/>
-      </geometry>
-      <material name="demo_chassis_grey"/>
-    </visual>
-    <collision>
-      <origin xyz="0 0 0" rpy="0 0 0"/>
-      <geometry>
-        <box size="${chassis_length} ${chassis_width} ${chassis_height}"/>
-      </geometry>
-    </collision>
-    <xacro:box_inertia mass="${chassis_mass}"
-                       x="${chassis_length}" y="${chassis_width}" z="${chassis_height}"/>
-  </link>
-  <!-- base_link sits one wheel-radius above the ground plane. -->
-  <joint name="base_footprint_joint" type="fixed">
-    <parent link="base_footprint"/>
-    <child link="base_link"/>
-    <origin xyz="0 0 ${wheel_radius}" rpy="0 0 0"/>
-  </joint>
-  <xacro:drive_wheel prefix="left"  y_offset="${ wheel_separation/2}"
-                     x_offset="${wheel_base_offset_x}"
-                     radius="${wheel_radius}" length="${wheel_width}" mass="${wheel_mass}"/>
-  <xacro:drive_wheel prefix="right" y_offset="${-wheel_separation/2}"
-                     x_offset="${wheel_base_offset_x}"
-                     radius="${wheel_radius}" length="${wheel_width}" mass="${wheel_mass}"/>
-  <!-- Caster hangs below base_link so its lowest point touches the floor
-       alongside the wheels: z = -(wheel_radius - caster_radius). -->
-  <xacro:caster_wheel x_offset="${chassis_length/2 - caster_radius*2}"
-                      z_offset="${-(wheel_radius - caster_radius)}"
-                      radius="${caster_radius}" mass="${caster_mass}"/>
-  <xacro:lidar_sensor x_offset="${lidar_offset_x}" z_offset="${lidar_offset_z}"
-                      size="0.03" mass="0.1" update_rate="10"
-                      samples="${lidar_samples}"
-                      range_min="0.12" range_max="${lidar_range_max}"
-                      gz_topic="scan"/>
-  <xacro:camera_sensor x_offset="${camera_offset_x}" z_offset="${camera_offset_z}"
-                       size="0.03" mass="0.1" update_rate="15"
-                       width="${camera_width}" height="${camera_height}"
-                       hfov="1.089"
-                       gz_topic="camera/image_raw"/>
-  <!-- ========================= Gazebo plugins ==========================
-       Inert in ML2 (RViz ignores <gazebo> tags); active from ML3 onward.
-       Chosen over gz_ros2_control deliberately: the native system plugin is
-       already present on the host and needs no ros2_control/controller_manager
-       stack. Swapping it later does not change /demo/cmd_vel, which is the
-       whole point of the topic contract. See plan decision 2.
+  <xacro:arg name="use_meshes" default="true"/>
+  <!--
+    The upstream model. Absolute-path include via $(find ...) so it resolves
+    through the ament share tree, not a relative path out of this package.
   -->
-  <gazebo>
-    <plugin filename="gz-sim-diff-drive-system" name="gz::sim::systems::DiffDrive">
-      <left_joint>left_wheel_joint</left_joint>
-      <right_joint>right_wheel_joint</right_joint>
-      <wheel_separation>${wheel_separation}</wheel_separation>
-      <wheel_radius>${wheel_radius}</wheel_radius>
-      <odom_publish_frequency>30</odom_publish_frequency>
-      <max_linear_acceleration>1.0</max_linear_acceleration>
-      <topic>cmd_vel</topic>
-      <odom_topic>odom</odom_topic>
-      <tf_topic>tf</tf_topic>
-      <frame_id>odom</frame_id>
-      <child_frame_id>base_footprint</child_frame_id>
-    </plugin>
-    <!-- Publishes wheel joint angles so robot_state_publisher can animate the
-         wheel TFs. Without this, wheels render frozen even while the robot moves. -->
-    <plugin filename="gz-sim-joint-state-publisher-system"
-            name="gz::sim::systems::JointStatePublisher">
-      <topic>joint_states</topic>
-      <joint_name>left_wheel_joint</joint_name>
-      <joint_name>right_wheel_joint</joint_name>
-    </plugin>
-  </gazebo>
-  <!-- Wheel contact properties. Driven wheels need grip; without explicit mu
-       the robot slips and odometry diverges from ground truth. -->
-  <gazebo reference="left_wheel_link">
-    <mu1>1.0</mu1>
-    <mu2>1.0</mu2>
-  </gazebo>
-  <gazebo reference="right_wheel_link">
-    <mu1>1.0</mu1>
-    <mu2>1.0</mu2>
-  </gazebo>
-  <gazebo reference="caster_wheel_link">
-    <mu1>0.0</mu1>
-    <mu2>0.0</mu2>
-  </gazebo>
+  <xacro:include filename="$(find nav2_minimal_tb4_description)/urdf/standard/turtlebot4.urdf.xacro"/>
+  <!--
+    ############################################################################
+    #  REQUIRED POST-PROCESSING — THE ROBOT FALLS APART WITHOUT IT             #
+    ############################################################################
+    Upstream tags 21 of its fixed joints with
+        <gazebo reference="..."><preserveFixedJoint>true</preserveFixedJoint></gazebo>
+    which tells Gazebo NOT to weld the joint's child into its parent's rigid body.
+    Spawned as-is, this robot is 13 INDEPENDENT PHYSICS BODIES (shell, four tower
+    standoffs, sensor plate, lidar, camera, bumper, wheels, caster, base) held
+    together only by fixed-joint constraints. The solver does not hold them
+    rigidly: under gravity and contact the parts settle and drift, the tower leans,
+    and the plate and lidar float off the standoffs.
+    That is the long-standing "robot with expanded/scattered parts" symptom, and it
+    is NOT a geometry bug — the offsets and per-visual rpy rotations here are
+    correct. Welding changes nothing about where parts are DRAWN, only whether
+    physics may move them relative to each other. Re-measuring mesh offsets and
+    swapping the robot model both failed to fix it for exactly this reason.
+    xacro CANNOT remove a tag that an include emits, so the strip happens in the
+    pipeline that feeds Gazebo:
+        xacro demo_robot.urdf.xacro | scripts/weld_fixed_joints.py > robot.urdf
+    demo_simulation/launch/simulation.launch.py does this. If you spawn this xacro
+    by any other route, pipe it through that script too, or the robot comes apart.
+    RViz2 is unaffected — it ignores <gazebo> blocks entirely and always draws the
+    assembled robot. So the model looks perfect in RViz and falls apart in Gazebo,
+    which is what makes this hard to attribute.
+  -->
+  <!--
+    ===================== Inherited from upstream, unchanged =====================
+    Deliberately NOT re-declared here (see note 2 in the file header — xacro
+    concatenates <gazebo> blocks instead of overriding them, so re-declaring any
+    of these produces a duplicate plugin rather than a replacement):
+      DiffDrive              gz topics /cmd_vel, /odom, tf; odom -> base_link;
+                             wheel_separation 0.233, wheel_radius 0.03575;
+                             clamps 0.5 m/s and 2.0 rad/s
+      JointStatePublisher    /joint_states for left_wheel_joint, right_wheel_joint
+      RPLIDAR A1             gz /scan, 360 samples, 10 Hz, frame rplidar_link
+      OAK-D RGBD             gz /rgbd_camera/{image,depth_image,points,camera_info}
+      IMU                    gz /imu at 200 Hz
+    wheel_separation and wheel_radius are the two values that must never drift
+    from the physical model: the plugin integrates them into odometry, so a
+    mismatch produces a robot that slides while reporting a straight line, with no
+    error anywhere. Inheriting them keeps them locked to the meshes by definition.
+    The IMU only publishes if the WORLD loads gz-sim-imu-system. The bundled
+    nav2_minimal_tb4_sim warehouse.sdf does; a hand-written world may not, and the
+    sensor then stays silent with no error. Verify with `gz topic -l | grep imu`.
+    All gz topic names above are literal/unscoped, which is what
+    demo_simulation/config/bridge_warehouse.yaml binds to. Gazebo also advertises
+    /model/<name>/* lookalikes with no publisher behind them; bridging to those
+    yields a robot that never moves, silently. See the long note in that file.
+  -->
 </robot>
